Commit message: feat: complete Phase 2 and 4 (pick/place and task manager)

File: src/robot1_moveit_config/srdf/ur_macro.srdf.xacro (robot description, xacro)
@@ -53,4 +53,31 @@
     <disable_collisions link1="${prefix}wrist_1_link" link2="${prefix}wrist_3_link" reason="Never" />
     <disable_collisions link1="${prefix}wrist_2_link" link2="${prefix}wrist_3_link" reason="Adjacent" />
-  </xacro:macro>
+    <!-- GRIPPER GROUP -->
+    <group name="robot1_gripper">
+      <joint name="robot1_robotiq_base_joint"/>
+      <joint name="robot1_robotiq_140_base_joint"/>
+      <joint name="robot1_finger_joint"/>
+      <joint name="robot1_left_inner_knuckle_joint"/>
+      <joint name="robot1_left_inner_finger_joint"/>
+      <joint name="robot1_right_outer_knuckle_joint"/>
+      <joint name="robot1_right_inner_knuckle_joint"/>
+      <joint name="robot1_right_inner_finger_joint"/>
+    </group>
+    <!-- END EFFECTOR -->
+    <end_effector name="robot1_gripper" parent_link="robot1_tool0" group="robot1_gripper" parent_group="robot1_ur_manipulator"/>
+    <!-- DISABLE COLLISIONS FOR GRIPPER -->
+    <disable_collisions link1="robot1_wrist_3_link" link2="robot1_robotiq_base_link" reason="Adjacent" />
+    <disable_collisions link1="robot1_wrist_3_link" link2="robot1_robotiq_140_base_link" reason="Default" />
+    <disable_collisions link1="robot1_robotiq_base_link" link2="robot1_robotiq_140_base_link" reason="Adjacent" />
+    <disable_collisions link1="robot1_robotiq_140_base_link" link2="robot1_left_outer_knuckle" reason="Adjacent" />
+    <disable_collisions link1="robot1_robotiq_140_base_link" link2="robot1_right_outer_knuckle" reason="Adjacent" />
+    <disable_collisions link1="robot1_robotiq_140_base_link" link2="robot1_left_inner_knuckle" reason="Adjacent" />
+    <disable_collisions link1="robot1_robotiq_140_base_link" link2="robot1_right_inner_knuckle" reason="Adjacent" />
+    <disable_collisions link1="robot1_left_outer_knuckle" link2="robot1_left_outer_finger" reason="Adjacent" />
+    <disable_collisions link1="robot1_right_outer_knuckle" link2="robot1_right_outer_finger" reason="Adjacent" />
+    <disable_collisions link1="robot1_left_inner_knuckle" link2="robot1_left_inner_finger" reason="Adjacent" />
+    <disable_collisions link1="robot1_right_inner_knuckle" link2="robot1_right_inner_finger" reason="Adjacent" />
+    <disable_collisions link1="robot1_left_outer_finger" link2="robot1_left_inner_finger" reason="Default" />
+    <disable_collisions link1="robot1_right_outer_finger" link2="robot1_right_inner_finger" reason="Default" />
+</xacro:macro>
 </robot>

File: src/robot2_moveit_config/srdf/ur_macro.srdf.xacro (robot description, xacro)
@@ -53,4 +53,31 @@
     <disable_collisions link1="${prefix}wrist_1_link" link2="${prefix}wrist_3_link" reason="Never" />
     <disable_collisions link1="${prefix}wrist_2_link" link2="${prefix}wrist_3_link" reason="Adjacent" />
-  </xacro:macro>
+    <!-- GRIPPER GROUP -->
+    <group name="robot2_gripper">
+      <joint name="robot2_robotiq_base_joint"/>
+      <joint name="robot2_robotiq_140_base_joint"/>
+      <joint name="robot2_finger_joint"/>
+      <joint name="robot2_left_inner_knuckle_joint"/>
+      <joint name="robot2_left_inner_finger_joint"/>
+      <joint name="robot2_right_outer_knuckle_joint"/>
+      <joint name="robot2_right_inner_knuckle_joint"/>
+      <joint name="robot2_right_inner_finger_joint"/>
+    </group>
+    <!-- END EFFECTOR -->
+    <end_effector name="robot2_gripper" parent_link="robot2_tool0" group="robot2_gripper" parent_group="robot2_ur_manipulator"/>
+    <!-- DISABLE COLLISIONS FOR GRIPPER -->
+    <disable_collisions link1="robot2_wrist_3_link" link2="robot2_robotiq_base_link" reason="Adjacent" />
+    <disable_collisions link1="robot2_wrist_3_link" link2="robot2_robotiq_140_base_link" reason="Default" />
+    <disable_collisions link1="robot2_robotiq_base_link" link2="robot2_robotiq_140_base_link" reason="Adjacent" />
+    <disable_collisions link1="robot2_robotiq_140_base_link" link2="robot2_left_outer_knuckle" reason="Adjacent" />
+    <disable_collisions link1="robot2_robotiq_140_base_link" link2="robot2_right_outer_knuckle" reason="Adjacent" />
+    <disable_collisions link1="robot2_robotiq_140_base_link" link2="robot2_left_inner_knuckle" reason="Adjacent" />
+    <disable_collisions link1="robot2_robotiq_140_base_link" link2="robot2_right_inner_knuckle" reason="Adjacent" />
+    <disable_collisions link1="robot2_left_outer_knuckle" link2="robot2_left_outer_finger" reason="Adjacent" />
+    <disable_collisions link1="robot2_right_outer_knuckle" link2="robot2_right_outer_finger" reason="Adjacent" />
+    <disable_collisions link1="robot2_left_inner_knuckle" link2="robot2_left_inner_finger" reason="Adjacent" />
+    <disable_collisions link1="robot2_right_inner_knuckle" link2="robot2_right_inner_finger" reason="Adjacent" />
+    <disable_collisions link1="robot2_left_outer_finger" link2="robot2_left_inner_finger" reason="Default" />
+    <disable_collisions link1="robot2_right_outer_finger" link2="robot2_right_inner_finger" reason="Default" />
+</xacro:macro>
 </robot>

File: src/robot3_moveit_config/srdf/ur_macro.srdf.xacro (robot description, xacro)
@@ -53,4 +53,31 @@
     <disable_collisions link1="${prefix}wrist_1_link" link2="${prefix}wrist_3_link" reason="Never" />
     <disable_collisions link1="${prefix}wrist_2_link" link2="${prefix}wrist_3_link" reason="Adjacent" />
-  </xacro:macro>
+    <!-- GRIPPER GROUP -->
+    <group name="robot3_gripper">
+      <joint name="robot3_robotiq_base_joint"/>
+      <joint name="robot3_robotiq_140_base_joint"/>
+      <joint name="robot3_finger_joint"/>
+      <joint name="robot3_left_inner_knuckle_joint"/>
+      <joint name="robot3_left_inner_finger_joint"/>
+      <joint name="robot3_right_outer_knuckle_joint"/>
+      <joint name="robot3_right_inner_knuckle_joint"/>
+      <joint name="robot3_right_inner_finger_joint"/>
+    </group>
+    <!-- END EFFECTOR -->
+    <end_effector name="robot3_gripper" parent_link="robot3_tool0" group="robot3_gripper" parent_group="robot3_ur_manipulator"/>
+    <!-- DISABLE COLLISIONS FOR GRIPPER -->
+    <disable_collisions link1="robot3_wrist_3_link" link2="robot3_robotiq_base_link" reason="Adjacent" />
+    <disable_collisions link1="robot3_wrist_3_link" link2="robot3_robotiq_140_base_link" reason="Default" />
+    <disable_collisions link1="robot3_robotiq_base_link" link2="robot3_robotiq_140_base_link" reason="Adjacent" />
+    <disable_collisions link1="robot3_robotiq_140_base_link" link2="robot3_left_outer_knuckle" reason="Adjacent" />
+    <disable_collisions link1="robot3_robotiq_140_base_link" link2="robot3_right_outer_knuckle" reason="Adjacent" />
+    <disable_collisions link1="robot3_robotiq_140_base_link" link2="robot3_left_inner_knuckle" reason="Adjacent" />
+    <disable_collisions link1="robot3_robotiq_140_base_link" link2="robot3_right_inner_knuckle" reason="Adjacent" />
+    <disable_collisions link1="robot3_left_outer_knuckle" link2="robot3_left_outer_finger" reason="Adjacent" />
+    <disable_collisions link1="robot3_right_outer_knuckle" link2="robot3_right_outer_finger" reason="Adjacent" />
+    <disable_collisions link1="robot3_left_inner_knuckle" link2="robot3_left_inner_finger" reason="Adjacent" />
+    <disable_collisions link1="robot3_right_inner_knuckle" link2="robot3_right_inner_finger" reason="Adjacent" />
+    <disable_collisions link1="robot3_left_outer_finger" link2="robot3_left_inner_finger" reason="Default" />
+    <disable_collisions link1="robot3_right_outer_finger" link2="robot3_right_inner_finger" reason="Default" />
+</xacro:macro>
 </robot>
